File: pcb/pcb.kicad_pcb (KiCad board)
At the start: 2 copper layers, 75.2 x 62.6 mm, 39 parts, among them J1 Conn_01x06, U1 ATmega328P-AU, U2 SRV05-4

Commit message: update
Parts:
- removed the D8 at (144.4, 75.7)
- added D4: D_Small, custom_parts:D_SOT-23_ANK, B.Cu at (144.4, 75.7)
- renumbered BOOT1 to BOOT, D2 to D1, D4 to D2, D6 to D3, D10 to D5, D12 to D6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
