File: pcb/pcb.sch (KiCad schematic (older format))
At the start: 39 parts, among them J1 Conn_01x06, U1 ATmega328P-AU, U2 SRV05-4

Commit message: add readme and fabrication files
Parts:
- BOOT1, RESET1: LCSC C318884 -> C318884
- C7, C8: LCSC C1804 -> C1804
- U1: LCSC C14877 -> C14877
Changed lines of the file:
@@
 F 2 "Capacitor_SMD:C_0805_2012Metric" H 5800 8050 50  0001 C CNN
 F 3 "~" H 5800 8050 50  0001 C CNN
-F 4 " C1804" V 5800 8050 50  0001 C CNN "LCSC"
+F 4 "C1804" V 5800 8050 50  0001 C CNN "LCSC"
 	1    5800 8050
 	0    -1   -1   0
@@
 F 2 "Capacitor_SMD:C_0805_2012Metric" H 5800 7700 50  0001 C CNN
 F 3 "~" H 5800 7700 50  0001 C CNN
-F 4 " C1804" V 5800 7700 50  0001 C CNN "LCSC"
+F 4 "C1804" V 5800 7700 50  0001 C CNN "LCSC"
 	1    5800 7700
 	0    -1   -1   0
@@
 F 2 "random-keyboard-parts:SKQG-1155865" H 1650 8000 50  0001 C CNN
 F 3 "~" H 1650 8000 50  0001 C CNN
-F 4 " C318884" H 1650 7800 50  0001 C CNN "LCSC"
+F 4 "C318884" H 1650 7800 50  0001 C CNN "LCSC"
 	1    1650 7800
 	1    0    0    -1
@@
 F 2 "Package_QFP:TQFP-32_7x7mm_P0.8mm" H 3850 8400 50  0001 C CIN
 F 3 "http://ww1.microchip.com/downloads/en/DeviceDoc/ATmega328_P%20AVR%20MCU%20with%20picoPower%20Technology%20Data%20Sheet%2040001984A.pdf" H 3850 8400 50  0001 C CNN
-F 4 " C14877" H 3850 8400 50  0001 C CNN "LCSC"
+F 4 "C14877" H 3850 8400 50  0001 C CNN "LCSC"
 	1    3850 8400
 	1    0    0    -1
@@
 F 2 "random-keyboard-parts:SKQG-1155865" H 1650 8700 50  0001 C CNN
 F 3 "~" H 1650 8700 50  0001 C CNN
-F 4 " C318884" H 1650 8500 50  0001 C CNN "LCSC"
+F 4 "C318884" H 1650 8500 50  0001 C CNN "LCSC"
 	1    1650 8500
 	1    0    0    -1

Commit message: update
Parts:
- renumbered D2 to D1, D4 to D2, D6 to D3, D8 to D4, D10 to D5, D12 to D6, D81 to D7, D82 to D8, XTAL1 to X1
Changed lines of the file:
@@
 	1450 10000 1600 10000
 $Comp
-L Device:Crystal_GND24_Small XTAL1
+L Device:Crystal_GND24_Small X1
 U 1 1 5FE3EF08
 P 5550 7900
-F 0 "XTAL1" V 5504 8044 50  0000 L CNN
+F 0 "X1" V 5504 8044 50  0000 L CNN
 F 1 "Crystal_GND24_Small" V 5595 8044 50  0000 L CNN
 F 2 "Crystal:Crystal_SMD_3225-4Pin_3.2x2.5mm" H 5550 7900 50  0001 C CNN
@@
 $EndComp
 $Comp
-L Device:D_Zener_Small D82
+L Device:D_Zener_Small D8
 U 1 1 60DD2FED
 P 8900 9850
-F 0 "D82" V 8854 9920 50  0000 L CNN
+F 0 "D8" V 8854 9920 50  0000 L CNN
 F 1 "D_Zener_Small" V 8945 9920 50  0000 L CNN
 F 2 "Diode_SMD:D_SOD-123" V 8900 9850 50  0001 C CNN
@@
 $EndComp
 $Comp
-L Device:D_Zener_Small D81
+L Device:D_Zener_Small D7
 U 1 1 60DD4FB7
 P 8650 9850
-F 0 "D81" V 8604 9920 50  0000 L CNN
+F 0 "D7" V 8604 9920 50  0000 L CNN
 F 1 "D_Zener_Small" V 8695 9920 50  0000 L CNN
 F 2 "Diode_SMD:D_SOD-123" V 8650 9850 50  0001 C CNN
@@
 	8500 5100 8350 5100
 $Comp
-L Device:D_Small D6
+L Device:D_Small D3
 U 1 1 5FEB901B
 P 8350 5200
-F 0 "D6" V 8396 5130 50  0000 R CNN
+F 0 "D3" V 8396 5130 50  0000 R CNN
 F 1 "D_Small" V 8305 5130 50  0000 R CNN
 F 2 "custom_parts:D_SOT-23_ANK" V 8350 5200 50  0001 C CNN
@@
 	8500 4400 8350 4400
 $Comp
-L Device:D_Small D2
+L Device:D_Small D1
 U 1 1 5FE9D2AE
 P 8350 4500
-F 0 "D2" V 8396 4430 50  0000 R CNN
+F 0 "D1" V 8396 4430 50  0000 R CNN
 F 1 "D_Small" V 8305 4430 50  0000 R CNN
 F 2 "custom_parts:D_SOT-23_ANK" V 8350 4500 50  0001 C CNN
@@
 	9800 3850 9800 4200
 $Comp
-L Device:D_Small D4
+L Device:D_Small D2
 U 1 1 5FE9EDA4
 P 9450 4500
-F 0 "D4" V 9496 4430 50  0000 R CNN
+F 0 "D2" V 9496 4430 50  0000 R CNN
 F 1 "D_Small" V 9405 4430 50  0000 R CNN
 F 2 "custom_parts:D_SOT-23_ANK" V 9450 4500 50  0001 C CNN
@@
 $EndComp
 $Comp
-L Device:D_Small D8
+L Device:D_Small D4
 U 1 1 5FEB9045
 P 9450 5200
-F 0 "D8" V 9496 5130 50  0000 R CNN
+F 0 "D4" V 9496 5130 50  0000 R CNN
 F 1 "D_Small" V 9405 5130 50  0000 R CNN
 F 2 "custom_parts:D_SOT-23_ANK" V 9450 5200 50  0001 C CNN
@@
 	8500 5800 8350 5800
 $Comp
-L Device:D_Small D10
+L Device:D_Small D5
 U 1 1 5FF3E804
 P 8350 5900
-F 0 "D10" V 8396 5830 50  0000 R CNN
+F 0 "D5" V 8396 5830 50  0000 R CNN
 F 1 "D_Small" V 8305 5830 50  0000 R CNN
 F 2 "custom_parts:D_SOT-23_ANK" V 8350 5900 50  0001 C CNN
@@
 $EndComp
 $Comp
-L Device:D_Small D12
+L Device:D_Small D6
 U 1 1 5FF3E839
 P 9450 5900
-F 0 "D12" V 9496 5830 50  0000 R CNN
+F 0 "D6" V 9496 5830 50  0000 R CNN
 F 1 "D_Small" V 9405 5830 50  0000 R CNN
 F 2 "custom_parts:D_SOT-23_ANK" V 9450 5900 50  0001 C CNN
